File: PCB/FPGA_DENDY.sch (EAGLE design)
At the start: 159 parts, among them CN1 DENDY60PINSLOT, J9 BYPASS, Q1 14.318 MHz, Q2 17.734 MHz, SW1 TL36PO, U1 SN74LVC8T245, U10 OPA2134U, U11 SN74LVC2G34DBVR, U12 SN74LVC2G04DBVR, U13 74LS373WMSO20, U2 SN74LVCH16T245DGGR, U3 SN74LVCH16T245DGGR, U4 EP2C5T144, U5 EPCS4, U6 SN74LVC541A, U7 THS7374IPWR, U8 SN74LVC2G34DBVR, U9 74LVC1G04GV, X1 057-010-1

Commit message: Add files via upload
Parts:
- added U14: SN74LVC2G34DBVR, SN74LVC2G34DBVR:SN74LVC2G34DBVR
Connections:
- removed net /ROMSEL_FPGA: CN1./ROMSEL
- new net /ROMSEL: CN1./ROMSEL, U14.OUT1
- new net R/W_FPGA: U14.IN2
- net +3V3: now also U14.VCC
- net /RS_FPGA: now also U14.IN1
- net GND: now also U14.GND
- net R/W: now also U14.OUT2
Other:
- moved on the sheet: C31, R27, U11, U12, U8

Commit message: Add files via upload
Parts:
- added C61, C62: 0.1uF, rcl_my:C-EUC0805
- added RN14: 8k2, resistor-dil:4R-N0603-ARC
- added X2, X4: (no value), con-subd:F15HPS
Connections:
- net +5V: now also C61.1, C62.1, RN14A.1, RN14B.1, RN14C.1, RN14D.1, X2-15.F, X4-15.F
- net GND: now also C61.2, C62.2, X2-1.F, X2-G.G1, X4-1.F, X4-G.G1
- net JOYDATA1: now also RN14A.2, X2-8.F
- net JOYDATA2: now also RN14B.2, X4-8.F
- net LE: now also X2-12.F, X4-12.F
- net SCK1: now also RN14C.2, X2-9.F
- net SCK2: now also RN14D.2, X4-9.F
Other:
- note added: "JOYPAD 1"
- note added: "JOYPAD 2"
- moved on the sheet: C59, C60, CN1
