File: PCB/FPGA_DENDY.sch (EAGLE design)
At the start: 165 parts, among them CN1 DENDY60PINSLOT, J9 BYPASS, Q1 14.318 MHz, Q2 17.734 MHz, SW1 TL36PO, U1 SN74LVC8T245, U10 OPA2134U, U11 SN74LVC2G34DBVR, U12 SN74LVC2G04DBVR, U13 74LS373WMSO20, U14 SN74LVC2G34DBVR, U2 SN74LVCH16T245DGGR, U3 SN74LVCH16T245DGGR, U4 EP2C5T144, U5 EPCS4, U6 SN74LVC541A, U7 THS7374IPWR, U8 SN74LVC2G34DBVR, U9 74LVC1G04GV, X1 057-010-1

Commit message: Add files via upload
Connections:
- removed net DATAO: U4.DATA0, U5.ASDI
- new net DATA0: U4.DATA0, U5.DATA
- net ASDO: now also U5.ASDI; no longer U5.DATA
Changed lines of the file:
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@@
 <?xml version="1.0" encoding="utf-8"?>
 <!DOCTYPE eagle SYSTEM "eagle.dtd">
-<eagle version="9.6.2">
+<eagle version="9.4.2">
 <drawing>
 <settings>
@@
 <setting verticaltext="up"/>
 </settings>
-<grid distance="0.1" unitdist="inch" unit="inch" style="lines" multiple="1" display="yes" altdistance="0.01" altunitdist="inch" altunit="inch"/>
+<grid distance="0.1" unitdist="inch" unit="inch" style="lines" multiple="1" display="no" altdistance="0.01" altunitdist="inch" altunit="inch"/>
 <layers>
 <layer number="1" name="Top" color="4" fill="1" visible="no" active="no"/>
@@
 <net name="ASDO" class="0">
 <segment>
-<wire x1="170.18" y1="2.54" x2="157.48" y2="2.54" width="0.1524" layer="91"/>
-<label x="157.48" y="2.54" size="1.778" layer="95"/>
-<pinref part="U5" gate="G$1" pin="DATA"/>
-</segment>
-<segment>
 <wire x1="-2.54" y1="73.66" x2="-15.24" y2="73.66" width="0.1524" layer="91"/>
 <label x="-10.16" y="73.66" size="1.778" layer="95"/>
 <pinref part="U4" gate="G$1" pin="IO1(ASDO)"/>
 </segment>
+<segment>
+<wire x1="203.2" y1="-2.54" x2="195.58" y2="-2.54" width="0.1524" layer="91"/>
+<label x="195.58" y="-2.54" size="1.778" layer="95"/>
+<pinref part="U5" gate="G$1" pin="ASDI"/>
+</segment>
 </net>
 <net name="/CSO" class="0">
@@
 </segment>
 </net>
-<net name="DATAO" class="0">
-<segment>
-<wire x1="195.58" y1="-2.54" x2="203.2" y2="-2.54" width="0.1524" layer="91"/>
-<label x="195.58" y="-2.54" size="1.778" layer="95"/>
-<pinref part="U5" gate="G$1" pin="ASDI"/>
-</segment>
+<net name="DATA0" class="0">
 <segment>
 <wire x1="132.08" y1="27.94" x2="142.24" y2="27.94" width="0.1524" layer="91"/>
@@
 <pinref part="U4" gate="G$1" pin="DATA0"/>
 </segment>
+<segment>
+<wire x1="157.48" y1="2.54" x2="170.18" y2="2.54" width="0.1524" layer="91"/>
+<label x="157.48" y="2.54" size="1.778" layer="95"/>
+<pinref part="U5" gate="G$1" pin="DATA"/>
+</segment>
 </net>
