File: PCB/Lattice PCB/FPGA_DENDY_LAT.sch (EAGLE design)
At the start: 165 parts, among them CN1 DENDY60PINSLOT, J9 BYPASS, Q1 14.318 MHz, Q2 17.734 MHz, U1 SN74LVC8T245, U10 OPA2134U, U11 SN74LVC2G34DBVR, U12 SN74LVC2G04DBVR, U13 74LS373WMSO20, U14 SN74LVC2G34DBVR, U15 SN74LVC1G240DCKR, U16 SN74LVC1G240DCKR, U17 SN74LVC1G125DBVR, U2 SN74LVCH16T245DGGR, U3 SN74LVCH16T245DGGR, U4 LCMXO2-4000HC-4TG144C, U5 SN74LVC1G240DCKR, U6 SN74LVC1G240DCKR, U7 THS7374IPWR, U9 74LVC1G04GV, X1 057-010-1, X2 JOYPAD1, X3 9V, X4 JOYPAD2

Commit message: Add files via upload
Parts:
- removed U16: SN74LVC1G240DCKR, SN74LVC1G240DCKR:SN74LVC1G240DCKR
- added U8: 74LS373WMSO20, 74LS373WM:74LS373WMSO20
- U13: value 74LS373WMSO20 -> SN74LVC1G240DBVR; device 74LS373WM:74LS373WMSO20 -> SN74LVC1G240DBVR:SN74LVC1G240DBVR
- U15, U5, U6: value SN74LVC1G240DCKR -> SN74LVC1G240DBVR; device SN74LVC1G240DCKR:SN74LVC1G240DCKR -> SN74LVC1G240DBVR:SN74LVC1G240DBVR
Connections:
- net +5V: now also U8.VCC; no longer U16.VCC
- net /IN0: now also U13./OE, U6./OE; no longer U15./OE, U5./OE
- net /IN1: now also U15./OE, U5./OE; no longer U16./OE, U6./OE
- net D0: now also U6.Y; no longer U16.Y
- net GND: now also U8./OE, U8.GND; no longer U13./OE, U16.GND
- net JOYDATA1: now also U6.A; no longer U15.A
- net JOYDATA2: now also U15.A; no longer U16.A
- net M2_JOY: now also U13.A; no longer U6.A
- net N$52: now also U8.EN; no longer U13.EN
- net PA0: now also U8.Q8; no longer U13.Q8
- net PA1: now also U8.Q6; no longer U13.Q6
- net PA2: now also U8.Q4; no longer U13.Q4
- net PA3: now also U8.Q2; no longer U13.Q2
- net PA4: now also U8.Q1; no longer U13.Q1
- net PA5: now also U8.Q3; no longer U13.Q3
- net PA6: now also U8.Q5; no longer U13.Q5
- net PA7: now also U8.Q7; no longer U13.Q7
- net PD0: now also U8.D8; no longer U13.D8
- net PD1: now also U8.D6; no longer U13.D6
- net PD2: now also U8.D4; no longer U13.D4
- net PD3: now also U8.D2; no longer U13.D2
- net PD4: now also U8.D1; no longer U13.D1
- net PD5: now also U8.D3; no longer U13.D3
- net PD6: now also U8.D5; no longer U13.D5
- net PD7: now also U8.D7; no longer U13.D7
- net SCK1: now also U13.Y; no longer U5.Y
- net SCK2: now also U5.Y; no longer U6.Y
Other:
- moved on the sheet: U15, U5, U6

Commit message: Add files via upload
Parts:
- removed C59, C61, C62: 0.1uF, rcl_my:C-EUC0805
- removed R62: 1k, rcl:R-EU_R0805
- removed U17: SN74LVC1G125DBVR, SN74LVC1G125DBVR:SN74LVC1G125DBVR
- added C28, C29, C30: 0.1uF, rcl_my:C-EUC0805
- added R31: 1k5, rcl:R-EU_R0805
- added U16: OPA2134U, burr-brown:OPA2134U
- C1, C8: device rcl_my:C-EUC0603 -> rcl_my:C-EUC0805
- C11: value 22uF -> 0.1uF; device rcl_my:C-EUC0603 -> rcl_my:C-EUC0805
- C14: value 0.1uF -> 1uF
- C31: value 1uF -> 100uF; device rcl_my:C-EUC0805 -> rcl_my:CPOL-EU153CLV-0505
- C36, C37: value 1000 -> 0.1uF
- C38: value 0.1uF -> 1000
- C39: value 10uF -> 0.1uF
- C4: value 100uF -> 0.1uF; device rcl_my:CPOL-EU153CLV-0505 -> rcl_my:C-EUC0805
- C40: value 10uF -> 1000
- C41: device rcl_my:C-EUC0805 -> rcl_my:C-EUC0603
- C42: value 0.1uF -> 22uF; device rcl_my:C-EUC0805 -> rcl_my:C-EUC0603
- C43: value 10uF -> 0.1uF; device rcl_my:CPOL-EU153CLV-0505 -> rcl_my:C-EUC0603
- C44: value 10uF -> 0.1uF; device rcl_my:CPOL-EU153CLV-0505 -> rcl_my:C-EUC0805
- C47, C51: value 0.1uF -> 10uF
- C49, C52: value 0.1uF -> 10uF; device rcl_my:C-EUC0805 -> rcl_my:CPOL-EU153CLV-0505
- R1: value 51 -> 10
- R10: value 1k -> 124
- R11: value 10 -> 287
- R12: value 4k7 -> 750
- R13: value 51 -> 124
- R14: value 750 -> 287
- R17: value 287 -> 1k
- R18, R21: value 124 -> 1k
- R19, R22: value 287 -> 2k
- R2, RN20: value 2k -> 4k7
- R20: value 750 -> 2k
- R23: value 4.7k -> 1k
- R24: value 75 -> 1k
- R26, R50: value 1.2k -> 1k
- R28: value 39k -> 2k2
- R29: value 20k -> 4k7
- R3: value 2k2 -> 4k7
- R30, RN15: value 4k7 -> 2k
- R32: value 1k -> 39k
- R33: value 2k -> 20k
- R34: value 4k7 -> 1,1k
- R35: value 2k -> 510
- R36: value 1k5 -> 10
- R4, R5: value 10k -> 1.2k
- R40: value 1,1k -> 75
- R41: value 510 -> 4.7k
- R42: value 2k -> 10k
- R43, R45: value 1k -> 10k
- R44: value 10 -> 10k
- R6, R7: value 10k -> 51
- R8: value 1k -> 287
- R9: value 1k -> 750
- RN1: value 2k -> 33
- RN10, RN14, RN16, RN4, RN7: value 2k -> 1k
- RN11, RN17, RN5, RN8: value 1k -> 2k
- RN12, RN13: value 33 -> 2k
- RN2: value 1k -> 33
- U1: value SN74LVC8T245 -> LCMXO2-4000HC-4TG144C; device SnapEDA-Library:SN74LVC8T245 -> LCMXO2-4000HC:LCMXO2-4000HC
- U10: value OPA2134U -> THS7374IPWR; device burr-brown:OPA2134U -> THS7374IPWR:THS7374IPWR
- U11: value SN74LVC2G34DBVR -> SN74LVC1G125DBVR; device SN74LVC2G34DBVR:SN74LVC2G34DBVR -> SN74LVC1G125DBVR:SN74LVC1G125DBVR
- U12: value SN74LVC2G04DBVR -> SN74LVC1G240DBVR; device SN74LVC2G04DBVR:SN74LVC2G04DBVR -> SN74LVC1G240DBVR:SN74LVC1G240DBVR
- U14: value SN74LVC2G34DBVR -> SN74LVC1G240DBVR; device SN74LVC2G34DBVR:SN74LVC2G34DBVR -> SN74LVC1G240DBVR:SN74LVC1G240DBVR
- U2: value SN74LVCH16T245DGGR -> 74LS373WMSO20; device SN74LVCH16T245DGGR:SN74LVCH16T245DGGR -> 74LS373WM:74LS373WMSO20
- U3: value SN74LVCH16T245DGGR -> SN74LVC8T245; device SN74LVCH16T245DGGR:SN74LVCH16T245DGGR -> SnapEDA-Library:SN74LVC8T245
- U4: value LCMXO2-4000HC-4TG144C -> SN74LVCH16T245DGGR; device LCMXO2-4000HC:LCMXO2-4000HC -> SN74LVCH16T245DGGR:SN74LVCH16T245DGGR
- U5: value SN74LVC1G240DBVR -> SN74LVCH16T245DGGR; device SN74LVC1G240DBVR:SN74LVC1G240DBVR -> SN74LVCH16T245DGGR:SN74LVCH16T245DGGR
- U6: value SN74LVC1G240DBVR -> 74LVC1G04GV; device SN74LVC1G240DBVR:SN74LVC1G240DBVR -> 74LVC1G04GV:74LVC1G04GV
- U7: value THS7374IPWR -> SN74LVC2G04DBVR; device THS7374IPWR:THS7374IPWR -> SN74LVC2G04DBVR:SN74LVC2G04DBVR
- U8: value 74LS373WMSO20 -> SN74LVC2G34DBVR; device 74LS373WM:74LS373WMSO20 -> SN74LVC2G34DBVR:SN74LVC2G34DBVR
- U9: value 74LVC1G04GV -> SN74LVC2G34DBVR; device 74LVC1G04GV:74LVC1G04GV -> SN74LVC2G34DBVR:SN74LVC2G34DBVR
- renumbered C60 to C13, R61 to R49, R63 to R46, R64 to R51, R65 to R47, R66 to R52, R67 to R48, R68 to R53
Connections:
- net #CS: now also R38.2; no longer R39.2
- net +5V: now also C12.2, C3.2, C33.1, C34.+, C35.1, C4.2, C42.2, C43.2, C44.1, C45.1, C5.2, C9.2, R3.1, R36.1, R41.1, R42.1, R43.1, R45.1, R5.2, U10.VS+, U11.VCC, U12.VCC, U2.VCC, U3.VCCB@1, U3.VCCB@2, U4.VCCA@1, U4.VCCA@2, U5.VCCA@1, U5.VCCA@2; no longer C11.2, C15.2, C32.1, C38.2, C4.+, C47.2, C5.1, C51.2, C52.2, C59.2, C61.1, C62.1, R12.1, R23.1, R4.1, R5.1, R50.2, R6.1, R7.1, U1.VCCB@1, U1.VCCB@2, U17.VCC, U2.VCCA@1, U2.VCCA@2, U3.VCCA@1, U3.VCCA@2, U5.VCC, U7.VS+, U9.VCC
- net /DENDY: now also U1.IO111; no longer U4.IO111
- net /IN0: now also U1.JTAGENB_IO97, U12./OE, U14./OE; no longer U13./OE, U4.JTAGENB_IO97, U6./OE
- net /IN1: now also U1.IO104, U13./OE; no longer U4.IO104, U5./OE
- net /IRQ: now also R3.2, U7.IN2; no longer R12.2, U12.IN2
- net /IRQ_FPGA: now also U1.IO32, U7.OUT2; no longer U12.OUT2, U4.IO32
- net /PA13: now also U6.OUT; no longer U9.OUT
- net /PAL: now also U1.IO110; no longer U4.IO110
- net /PRD: now also U5.2A1; no longer U3.2A1
- net /PRD_FPGA: now also U1.IO20, U5.2B1; no longer U3.2B1, U4.IO20
- net /PWR: now also U5.2A2; no longer U3.2A2
- net /PWR_FPGA: now also U1.IO19, U5.2B2; no longer U3.2B2, U4.IO19
- net /RESET: now also C14.2, R2.2, U7.IN1; no longer C31.2, R27.2, U12.IN1
- net /ROMSEL: now also U8.OUT1; no longer U14.OUT1
- net /RS_FPGA: now also U1.IO31, U8.IN1; no longer U14.IN1, U4.IO31
- net /VCS_FPGA: now also U1.IO11, U9.OUT1; no longer U11.OUT1, U4.IO11
- net 6502_T1: now also R4.2, U1.IO105; no longer R26.2, U4.IO105
- net A0: now also U4.2A8; no longer U2.2A8
- net A0_FPGA: now also U1.IO34, U4.2B8; no longer U2.2B8, U4.IO34
- net A1: now also U4.2A7; no longer U2.2A7
- net A10: now also U4.1A3; no longer U2.1A3
- net A10_FPGA: now also U1.IO47, U4.1B3; no longer U2.1B3, U4.IO47
- net A11: now also U4.1A1; no longer U2.1A1
- net A11_FPGA: now also U1.IO49, U4.1B1; no longer U2.1B1, U4.IO49
- net A12: now also U4.1A4; no longer U2.1A4
- net A12_FPGA: now also U1.IO46, U4.1B4; no longer U2.1B4, U4.IO46
- net A13: now also U4.1A6; no longer U2.1A6
- net A13_FPGA: now also U1.IO44_PCLKT2_1, U4.1B6; no longer U2.1B6, U4.IO44_PCLKT2_1
- net A14: now also U4.1A8; no longer U2.1A8
- net A14_FPGA: now also U1.IO42, U4.1B8; no longer U2.1B8, U4.IO42
- net A1_FPGA: now also U1.IO35, U4.2B7; no longer U2.2B7, U4.IO35
- net A2: now also U4.2A6; no longer U2.2A6
- net A2_FPGA: now also U1.IO36, U4.2B6; no longer U2.2B6, U4.IO36
- net A3: now also U4.2A5; no longer U2.2A5
- net A3_FPGA: now also U1.IO37, U4.2B5; no longer U2.2B5, U4.IO37
- net A4: now also U4.2A4; no longer U2.2A4
- net A4_FPGA: now also U1.IO38, U4.2B4; no longer U2.2B4, U4.IO38
- net A5: now also U4.2A3; no longer U2.2A3
- net A5_FPGA: now also U1.IO39, U4.2B3; no longer U2.2B3, U4.IO39
- net A6: now also U4.2A2; no longer U2.2A2
- net A6_FPGA: now also U1.IO40_PCLKT2_0, U4.2B2; no longer U2.2B2, U4.IO40_PCLKT2_0
- net A7: now also U4.2A1; no longer U2.2A1
- net A7_FPGA: now also U1.IO41_PCLKC2_0, U4.2B1; no longer U2.2B1, U4.IO41_PCLKC2_0
- net A8: now also U4.1A7; no longer U2.1A7
- net A8_FPGA: now also U1.IO43, U4.1B7; no longer U2.1B7, U4.IO43
- net A9: now also U4.1A5; no longer U2.1A5
- net A9_FPGA: now also U1.IO45_PCLKC2_1, U4.1B5; no longer U2.1B5, U4.IO45_PCLKC2_1
- net ALE: now also R1.1, U1.IO10; no longer R11.1, U4.IO10
- net B: now also R39.2; no longer R24.2
- net B0: now also RN5C.2, U1.IO80; no longer RN9C.2, U4.IO80
- net B1: now also RN5D.2, U1.IO81; no longer RN9D.2, U4.IO81
- net B2: now also RN3A.2, U1.IO82; no longer RN7A.2, U4.IO82
- net B3: now also RN3B.2, U1.IO83; no longer RN7B.2, U4.IO83
- net B4: now also RN3C.2, U1.IO84; no longer RN7C.2, U4.IO84
- net B5: now also RN3D.2, U1.IO85; no longer RN7D.2, U4.IO85
- net CLKN: now also R6.2, U1.PCLKT0_0_IO101; no longer R1.2, U4.PCLKT0_0_IO101
- net CLKP: now also R7.2, U1.PCLKT0_1_IO103; no longer R13.2, U4.PCLKT0_1_IO103
- net COMP0: now also RN12C.2, U1.IO94; no longer RN18C.2, U4.IO94
- net COMP1: now also RN12B.2, U1.IO93; no longer RN18B.2, U4.IO93
- net COMP2: now also RN12A.2, U1.IO92; no longer RN18A.2, U4.IO92
- net COMP3: now also RN13D.2, U1.IO91; no longer RN16D.2, U4.IO91
- net COMP4: now also RN13C.2, U1.IO90; no longer RN16C.2, U4.IO90
- net COMP5: now also RN13B.2, U1.IO89; no longer RN16B.2, U4.IO89
- net COMP6: now also RN13A.2, U1.IO88; no longer RN16A.2, U4.IO88
- net CO_DAC: now also R32.2, RN13A.1, RN14A.2; no longer R28.2, RN16A.1, RN17A.2
- net CS_FPGA: now also R34.2, U1.IO87; no longer R40.2, U4.IO87
- net D0: now also U14.Y, U5.1A8; no longer U3.1A8, U6.Y
- net D0_FPGA: now also U1.IO21, U5.1B8; no longer U3.1B8, U4.IO21
- net D1: now also U5.1A7; no longer U3.1A7
- net D1_FPGA: now also U1.IO22, U5.1B7; no longer U3.1B7, U4.IO22
- net D2: now also U5.1A6; no longer U3.1A6
- net D2_FPGA: now also U1.IO23_PCLKT3_0, U5.1B6; no longer U3.1B6, U4.IO23_PCLKT3_0
- net D3: now also U5.1A5; no longer U3.1A5
- net D3_FPGA: now also U1.IO24_PCLKC3_0, U5.1B5; no longer U3.1B5, U4.IO24_PCLKC3_0
- net D4: now also U5.1A4; no longer U3.1A4
- net D4_FPGA: now also U1.IO25, U5.1B4; no longer U3.1B4, U4.IO25
- net D5: now also U5.1A3; no longer U3.1A3
- net D5_FPGA: now also U1.IO26, U5.1B3; no longer U3.1B3, U4.IO26
- net D6: now also U5.1A2; no longer U3.1A2
- net D6_FPGA: now also U1.IO27, U5.1B2; no longer U3.1B2, U4.IO27
- net D7: now also U5.1A1; no longer U3.1A1
- net D7_FPGA: now also U1.IO28, U5.1B1; no longer U3.1B1, U4.IO28
- net DB_DIR: now also U1.IO29, U5.1DIR; no longer U3.1DIR, U4.IO29
- net DMC0: now also RN17C.2, U1.IO62; no longer RN20C.2, U4.IO62
- net DMC1: now also RN17B.2, U1.IO61; no longer RN20B.2, U4.IO61
- net DMC2: now also RN17A.2, U1.IO60; no longer RN20A.2, U4.IO60
- net DMC3: now also RN18D.2, U1.IO59; no longer RN14D.2, U4.IO59
- net DMC4: now also RN18C.2, U1.IO58; no longer RN14C.2, U4.IO58
- net DMC5: now also RN18B.2, U1.IO57; no longer RN14B.2, U4.IO57
- net DMC6: now also RN18A.2, U1.IO56; no longer RN14A.2, U4.IO56
- net DMC_DAC: now also R26.1, R30.1, RN18A.1; no longer R32.1, R35.1, RN14A.1
- net EMPH_B: now also R9.1, U1.IO86; no longer R15.1, U4.IO86
- net EMPH_G: now also R12.1, U1.IO79; no longer R14.1, U4.IO79
- net EMPH_R: now also R15.1, U1.IO72; no longer R20.1, U4.IO72
- net G0: now also RN8C.2, U1.PCLKC1_0_IO73; no longer RN6C.2, U4.PCLKC1_0_IO73
- net G1: now also RN8D.2, U1.PCLKT1_0_IO74; no longer RN6D.2, U4.PCLKT1_0_IO74
- net G2: now also RN6A.2, U1.IO75; no longer RN4A.2, U4.IO75
- net G3: now also RN6B.2, U1.IO76; no longer RN4B.2, U4.IO76
- net G4: now also RN6C.2, U1.IO77; no longer RN4C.2, U4.IO77
- net G5: now also RN6D.2, U1.IO78; no longer RN4D.2, U4.IO78
- net GND: now also C10.1, C12.1, C15.2, C16.1, C17.1, C18.1, C2.1, C20.1, C23.2, C25.2, C26.2, C27.2, C28.2, C29.2, C3.1, C30.2, C31.-, C35.2, C38.2, C39.2, C4.1, C40.2, C43.1, C44.2, C5.1, C50.2, C51.2, C6.1, C7.1, C9.1, R11.1, R14.1, R28.2, R33.1, R35.1, R50.2, R8.1, RN12D.2, RN17D.2, RN20A.1, RN20D.1, U1.GND@10, U1.GND@11, U1.GND@12, U1.GND@4, U1.GND@5, U1.GND@6, U1.GND@7, U1.GND@8, U1.GND@9, U10.DISABLE, U10.GND, U11./OE, U16A.V-, U2./OE, U2.GND, U3./OE, U4.1DIR, U4.2DIR, U5.2!OE, U5.2DIR, U5.GND@1, U5.GND@2, U5.GND@3, U5.GND@4, U5.GND@5, U5.GND@6, U5.GND@7, U5.GND@8; no longer C10.2, C12.2, C15.1, C16.2, C17.2, C18.2, C2.2, C20.2, C23.1, C25.1, C26.1, C27.1, C3.2, C31.1, C35.1, C38.1, C4.-, C46.2, C47.1, C49.1, C5.2, C50.1, C51.1, C52.1, C59.1, C6.2, C61.2, C62.2, C7.2, C9.2, R17.1, R19.1, R2.1, R29.1, R3.2, R41.1, R62.2, RN15A.1, RN15D.1, RN18D.2, RN20D.2, U1./OE, U10A.V-, U17./OE, U17.GND, U2.1DIR, U2.2DIR, U2.GND@1, U2.GND@2, U2.GND@3, U2.GND@4, U2.GND@5, U2.GND@6, U2.GND@7, U2.GND@8, U3.2!OE, U3.2DIR, U3.GND@4, U3.GND@5, U3.GND@6, U3.GND@7, U3.GND@8, U4.GND@10, U4.GND@11, U4.GND@12, U4.GND@9, U5.GND, U7.DISABLE, U8./OE
- net JOYDATA1: now also R42.2, U14.A; no longer R7.2, U6.A
- net JOYDATA2: now also R44.2; no longer R6.2
- net LCH: now also C52.-; no longer C44.-
- net LE: now also U11.Y; no longer U17.Y
- net LE_FPGA: now also U1.IO95, U11.A; no longer U17.A, U4.IO95
- net M2: now also U4.1A2; no longer U2.1A2
- net M2_FPGA: now also U1.IO48, U4.1B2; no longer U2.1B2, U4.IO48
- net M2_JOY: now also U1.PROGRAMN_IO96, U12.A; no longer U4.PROGRAMN_IO96, U5.A
- net N$1: now also C46.1, R25.2, R26.2, R27.2; no longer C39.1, R30.2, R32.2, R33.2
- net N$10: now also RN1B.2, U3.A1; no longer RN12B.2, U1.A1
- net N$11: now also RN13B.1, RN14A.1, RN14B.2; no longer RN16B.1, RN17A.1, RN17B.2
- net N$12: now also RN1C.2, U3.A2; no longer RN12C.2, U1.A2
- net N$13: now also RN1D.2, U3.A3; no longer RN12D.2, U1.A3
- net N$14: now also R10.1, R9.2, RN3D.1, RN4D.2; no longer R15.2, R16.1, RN7D.1, RN8D.2
- net N$15: now also U16B.-IN; no longer U10B.-IN
- net N$16: now also RN3C.1, RN4C.2, RN4D.1; no longer RN7C.1, RN8C.2, RN8D.1
- net N$17: now also RN2A.2, U3.A4; no longer RN13A.2, U1.A4
- net N$18: now also RN3B.1, RN4B.2, RN4C.1; no longer RN7B.1, RN8B.2, RN8C.1
- net N$19: now also R34.1, R35.2; no longer R40.1, R41.2
- net N$2: now also R7.1; no longer R13.1
- net N$20: now also RN13C.1, RN14B.1, RN14C.2; no longer RN16C.1, RN17B.1, RN17C.2
- net N$21: now also RN13D.1, RN14C.1, RN14D.2; no longer RN16D.1, RN17C.1, RN17D.2
- net N$22: now also R17.2, RN12C.1, RN12D.1; no longer R8.2, RN18C.1, RN18D.1
- net N$23: now also RN3A.1, RN4A.2, RN4B.1; no longer RN7A.1, RN8A.2, RN8B.1
- net N$24: now also R12.2, R13.1, RN6D.1, RN7D.2; no longer R14.2, R18.1, RN4D.1, RN5D.2
- net N$25: now also RN6C.1, RN7C.2, RN7D.1; no longer RN4C.1, RN5C.2, RN5D.1
- net N$26: now also RN6B.1, RN7B.2, RN7C.1; no longer RN4B.1, RN5B.2, RN5C.1
- net N$27: now also RN4A.1, RN5A.1, RN5B.1, RN5D.1; no longer RN8A.1, RN9A.1, RN9B.1, RN9D.1
- net N$28: now also RN6A.1, RN7A.2, RN7B.1; no longer RN4A.1, RN5A.2, RN5B.1
- net N$29: now also RN5A.2, RN5B.2, RN5C.1; no longer RN9A.2, RN9B.2, RN9C.1
- net N$30: now also C47.1, R29.2, R30.2, R31.2; no longer C40.1, R34.2, R35.2, R36.2
- net N$31: now also RN2B.2, U3.A5; no longer RN13B.2, U1.A5
- net N$32: now also RN2C.2, U3.A6; no longer RN13C.2, U1.A6
- net N$33: now also RN7A.1, RN8A.1, RN8B.1, RN8D.1; no longer RN5A.1, RN6A.1, RN6B.1, RN6D.1
- net N$34: now also R15.2, R16.1, RN10D.2, RN9D.1; no longer R20.2, R21.1, RN1D.1, RN2D.2
- net N$35: now also RN10C.2, RN10D.1, RN9C.1; no longer RN1C.1, RN2C.2, RN2D.1
- net N$36: now also RN8A.2, RN8B.2, RN8C.1; no longer RN6A.2, RN6B.2, RN6C.1
- net N$37: now also C49.+; no longer C43.+
- net N$38: now also R11.2, R13.2, U10.CH2_IN; no longer R18.2, R19.2, U7.CH2_IN
- net N$39: now also RN10B.2, RN10C.1, RN9B.1; no longer RN1B.1, RN2B.2, RN2C.1
- net N$4: now also C46.2, RN20C.1, RN20D.2, U16A.+IN; no longer C39.2, RN15C.1, RN15D.2, U10A.+IN
- net N$40: now also RN10A.2, RN10B.1, RN9A.1; no longer RN1A.1, RN2A.2, RN2B.1
- net N$41: now also RN10A.1, RN11A.1, RN11B.1, RN11D.1; no longer RN2A.1, RN3A.1, RN3B.1, RN3D.1
- net N$42: now also U16A.-IN; no longer U10A.-IN
- net N$43: now also U16A.OUT; no longer U10A.OUT
- net N$44: now also U16B.OUT; no longer U10B.OUT
- net N$45: now also C52.+; no longer C44.+
- net N$46: now also R18.1, RN12A.1, RN14D.1; no longer R9.1, RN17D.1, RN18A.1
- net N$47: now also R17.1, R18.2, RN12B.1; no longer R8.1, R9.2, RN18B.1
- net N$49: now also R32.1, R33.2; no longer R28.1, R29.2
- net N$5: now also RN18B.1; no longer RN14B.1
- net N$50: now also R36.2; no longer R44.2
- net N$52: now also R1.2, U2.EN; no longer R11.2, U8.EN
- net N$53: now also R14.2, R16.2, U10.CH3_IN; no longer R21.2, R22.2, U7.CH3_IN
- net N$54: now also R4.1; no longer R26.1
- net N$55: now also RN15D.1, RN16C.1, RN16D.2; no longer RN10D.1, RN11C.1, RN11D.2
- net N$56: now also R41.2, U10.BYPASS; no longer R23.2, U7.BYPASS
- net N$57: now also RN15C.1, RN16B.1, RN16C.2; no longer RN10C.1, RN11B.1, RN11C.2
- net N$58: now also R10.2, R8.2, U10.CH1_IN; no longer R16.2, R17.2, U7.CH1_IN
- net N$59: now also RN15B.1, RN16A.1, RN16B.2; no longer RN10B.1, RN11A.1, RN11B.2
- net N$6: now also R6.1; no longer R1.1
- net N$60: now also R22.2, RN15A.1, RN16A.2; no longer R2.2, RN10A.1, RN11A.2
- net N$61: now also RN2D.2, U3.A7; no longer RN13D.2, U1.A7
- net N$62: now also U10.CH4_IN; no longer U7.CH4_IN
- net N$63: now also R5.1; no longer R50.1
- net N$64: now also R39.1, U10.CH1_OUT; no longer R24.1, U7.CH1_OUT
- net N$65: now also U10.CH2_OUT; no longer U7.CH2_OUT
- net N$66: now also R40.1, U10.CH3_OUT; no longer R38.1, U7.CH3_OUT
- net N$67: now also R38.1, U10.CH4_OUT; no longer R39.1, U7.CH4_OUT
- net N$68: now also RN18C.1; no longer RN14C.1
- net N$69: now also RN18D.1; no longer RN14D.1
- net N$7: now also C47.2, RN20A.2, RN20B.1, U16B.+IN; no longer C40.2, RN15A.2, RN15B.1, U10B.+IN
- net N$70: now also R23.2, RN17C.1, RN17D.1; no longer R43.2, RN20C.1, RN20D.1
- net N$71: now also RN11A.2, RN11B.2, RN11C.1; no longer RN3A.2, RN3B.2, RN3C.1
- net N$72: now also R24.1, RN17A.1; no longer R45.1, RN20A.1
- net N$73: now also R23.1, R24.2, RN17B.1; no longer R43.1, R45.2, RN20B.1
- net N$8: now also R20.2, R21.1, RN16D.1; no longer R10.1, R42.2, RN11D.1
- net N$9: now also RN1A.2, U3.A0; no longer RN12A.2, U1.A0
- net PA0: now also U2.Q8; no longer U8.Q8
- net PA1: now also U2.Q6; no longer U8.Q6
- net PA10: now also U5.2A5; no longer U3.2A5
- net PA10_FPGA: now also U1.IO16_PCLKC4_0, U5.2B5; no longer U3.2B5, U4.IO16_PCLKC4_0
- net PA11: now also U5.2A6; no longer U3.2A6
- net PA11_FPGA: now also U1.IO15_PCLKT4_0, U5.2B6; no longer U3.2B6, U4.IO15_PCLKT4_0
- net PA12: now also U5.2A7; no longer U3.2A7
- net PA12_FPGA: now also U1.IO14, U5.2B7; no longer U3.2B7, U4.IO14
- net PA13: now also U5.2A8, U6.IN; no longer U3.2A8, U9.IN
- net PA13_FPGA: now also U1.IO13, U5.2B8; no longer U3.2B8, U4.IO13
- net PA2: now also U2.Q4; no longer U8.Q4
- net PA3: now also U2.Q2; no longer U8.Q2
- net PA4: now also U2.Q1; no longer U8.Q1
- net PA5: now also U2.Q3; no longer U8.Q3
- net PA6: now also U2.Q5; no longer U8.Q5
- net PA7: now also U2.Q7; no longer U8.Q7
- net PA8: now also U5.2A3; no longer U3.2A3
- net PA8_FPGA: now also U1.IO18, U5.2B3; no longer U3.2B3, U4.IO18
- net PA9: now also U5.2A4; no longer U3.2A4
- net PA9_FPGA: now also U1.IO17, U5.2B4; no longer U3.2B4, U4.IO17
- net PALSEL0: now also U1.PCLKC0_0_IO100; no longer U4.PCLKC0_0_IO100
- net PALSEL1: now also U1.IO99; no longer U4.IO99
- net PALSEL2: now also U1.IO98; no longer U4.IO98
- net PD0: now also U2.D8, U3.B0; no longer U1.B0, U8.D8
- net PD0_FPGA: now also RN1A.1, U1.IO8; no longer RN12A.1, U4.IO8
- net PD1: now also U2.D6, U3.B2; no longer U1.B2, U8.D6
- net PD1_FPGA: now also RN1C.1, U1.IO6_PCLKC5_0; no longer RN12C.1, U4.IO6_PCLKC5_0
- net PD2: now also U2.D4, U3.B4; no longer U1.B4, U8.D4
- net PD2_FPGA: now also RN2A.1, U1.IO4; no longer RN13A.1, U4.IO4
- net PD3: now also U2.D2, U3.B6; no longer U1.B6, U8.D2
- net PD3_FPGA: now also RN2C.1, U1.IO2; no longer RN13C.1, U4.IO2
- net PD4: now also U2.D1, U3.B7; no longer U1.B7, U8.D1
- net PD4_FPGA: now also RN2D.1, U1.IO1; no longer RN13D.1, U4.IO1
- net PD5: now also U2.D3, U3.B5; no longer U1.B5, U8.D3
- net PD5_FPGA: now also RN2B.1, U1.IO3; no longer RN13B.1, U4.IO3
- net PD6: now also U2.D5, U3.B3; no longer U1.B3, U8.D5
- net PD6_FPGA: now also RN1D.1, U1.IO5_PCLKT5_0; no longer RN12D.1, U4.IO5_PCLKT5_0
- net PD7: now also U2.D7, U3.B1; no longer U1.B1, U8.D7
- net PD7_FPGA: now also RN1B.1, U1.IO7; no longer RN12B.1, U4.IO7
- net PD_DIR: now also U1.IO9, U3.DIR; no longer U1.DIR, U4.IO9
- net R: now also R40.2; no longer R38.2
- net R/W: now also U8.OUT2; no longer U14.OUT2
- net R/W_FPGA: now also U1.IO30, U8.IN2; no longer U14.IN2, U4.IO30
- net R0: now also RN11C.2, U1.IO66; no longer RN3C.2, U4.IO66
- net R1: now also RN11D.2, U1.IO67; no longer RN3D.2, U4.IO67
- net R2: now also RN9A.2, U1.IO68; no longer RN1A.2, U4.IO68
- net R3: now also RN9B.2, U1.IO69; no longer RN1B.2, U4.IO69
- net R4: now also RN9C.2, U1.IO70; no longer RN1C.2, U4.IO70
- net R5: now also RN9D.2, U1.IO71; no longer RN1D.2, U4.IO71
- net RCH: now also C49.-; no longer C43.-
- net RESET: now also U1.IO33, U4.1!OE, U4.2!OE, U5.1!OE, U7.OUT1; no longer U12.OUT1, U2.1!OE, U2.2!OE, U3.1!OE, U4.IO33
- net SCK1: now also R43.2, U12.Y; no longer R4.2, U13.Y
- net SCK2: now also R45.2, U13.Y; no longer R5.2, U5.Y
- net SND: now also R25.1, R31.1; no longer R33.1, R36.1
- net SND0: now also RN15A.2, U1.IO50; no longer RN10A.2, U4.IO50
- net SND1: now also RN15B.2, U1.IO51; no longer RN10B.2, U4.IO51
- net SND2: now also RN15C.2, U1.IO52; no longer RN10C.2, U4.IO52
- net SND3: now also RN15D.2, U1.IO53; no longer RN10D.2, U4.IO53
- net SND4: now also R20.1, U1.IO54; no longer R42.1, U4.IO54
- net SND5: now also R19.1, U1.IO55; no longer R25.1, U4.IO55
- net SND_DAC: now also R19.2, R21.2; no longer R10.2, R25.2
- net SND_EXT: now also R27.1, R28.1, R29.1; no longer R3.1, R30.1, R34.1
- net TCK: now also U1.TCK; no longer U4.TCK
- net TDI: now also U1.TDI; no longer U4.TDI
- net TDO: now also U1.TDO; no longer U4.TDO
- net TMS: now also U1.TMS; no longer U4.TMS
- net VA10: now also U9.IN2; no longer U11.IN2
- net VA10_FPGA: now also U1.IO12, U9.OUT2; no longer U11.OUT2, U4.IO12
- net VCC: now also C31.+, C32.1, C48.2, RN20B.2, RN20C.2, U16A.V+; no longer C33.1, C34.+, C42.2, RN15B.2, RN15C.2, U10A.V+
- net VCCIO: now also C10.2, C11.2, C15.1, C16.2, C17.2, C18.2, C2.2, C20.2, C23.1, C25.1, C26.1, C27.1, C28.1, C29.1, C30.1, C38.1, C39.1, C40.1, C6.2, C7.2, R2.1, U1.VCC@1, U1.VCC@2, U1.VCC@3, U1.VCC@4, U1.VCCIO@0_1, U1.VCCIO@0_2, U1.VCCIO@0_3, U1.VCCIO@1_1, U1.VCCIO@1_2, U1.VCCIO@1_3, U1.VCCIO@2_1, U1.VCCIO@2_2, U1.VCCIO@2_3, U1.VCCIO@3, U1.VCCIO@4, U1.VCCIO@5, U3.VCCA, U4.VCCB@1, U4.VCCB@2, U5.VCCB@1, U5.VCCB@2, U7.VCC, U9.VCC; no longer C10.1, C12.1, C14.2, C16.1, C17.1, C18.1, C2.1, C20.1, C23.2, C25.2, C26.2, C27.2, C3.1, C35.2, C48.2, C49.2, C50.2, C6.1, C7.1, C9.1, R27.1, U1.VCCA, U11.VCC, U12.VCC, U2.VCCB@1, U2.VCCB@2, U3.VCCB@1, U3.VCCB@2, U4.VCC@1, U4.VCC@2, U4.VCC@3, U4.VCC@4, U4.VCCIO@0_1, U4.VCCIO@0_2, U4.VCCIO@0_3, U4.VCCIO@1_1, U4.VCCIO@1_2, U4.VCCIO@1_3, U4.VCCIO@2_1, U4.VCCIO@2_2, U4.VCCIO@2_3, U4.VCCIO@3, U4.VCCIO@4, U4.VCCIO@5
- net VPPL3: now also C50.1, C51.1, R50.1; no longer C45.1, C46.1, R62.1
- net VRAMSC: now also U9.IN1; no longer U11.IN1
Other:
- moved on the sheet: C1, C10, C11, C12, C14, C15, C16, C17, C18, C19, C2, C20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

Commit message: Add files via upload
Parts:
- renumbered Q1 to XO1, Q2 to XO2
Other:
- moved on the sheet: C34, C35, C36
