File: PCB/Lattice PCB/FPGA_DENDY_LAT.sch (EAGLE design)
At the start: 165 parts, among them CN1 DENDY60PINSLOT, J9 BYPASS, U1 LCMXO2-4000HC-4TG144C, U10 THS7374IPWR, U11 SN74LVC1G125DBVR, U12 SN74LVC1G240DBVR, U13 SN74LVC1G240DBVR, U14 SN74LVC1G240DBVR, U15 SN74LVC1G240DBVR, U16 OPA2134U, U2 74LS373WMSO20, U3 SN74LVC8T245, U4 SN74LVCH16T245DGGR, U5 SN74LVCH16T245DGGR, U6 74LVC1G04GV, U7 SN74LVC2G04DBVR, U8 SN74LVC2G34DBVR, U9 SN74LVC2G34DBVR, X1 057-010-1, X2 JOYPAD1, X3 9V, X4 JOYPAD2

Commit message: fix snd_dac wire
Connections:
- removed net SND: R25.1, R31.1
- net SND_DAC: now also R25.1, R31.1
Changed lines of the file:
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@@
 <junction x="182.88" y="-96.52"/>
+</segment>
+<segment>
+<wire x1="203.2" y1="-134.62" x2="220.98" y2="-134.62" width="0.1524" layer="91"/>
+<label x="205.74" y="-134.62" size="1.778" layer="95"/>
+<pinref part="R25" gate="G$1" pin="1"/>
+</segment>
+<segment>
+<wire x1="203.2" y1="-185.42" x2="220.98" y2="-185.42" width="0.1524" layer="91"/>
+<label x="205.74" y="-185.42" size="1.778" layer="95"/>
+<pinref part="R31" gate="G$1" pin="1"/>
 </segment>
 </net>
@@
 </segment>
 </net>
-<net name="SND" class="0">
-<segment>
-<wire x1="203.2" y1="-185.42" x2="220.98" y2="-185.42" width="0.1524" layer="91"/>
-<label x="205.74" y="-185.42" size="1.778" layer="95"/>
-<pinref part="R31" gate="G$1" pin="1"/>
-</segment>
-<segment>
-<wire x1="203.2" y1="-134.62" x2="220.98" y2="-134.62" width="0.1524" layer="91"/>
-<label x="205.74" y="-134.62" size="1.778" layer="95"/>
-<pinref part="R25" gate="G$1" pin="1"/>
-</segment>
-</net>
