File: PCB/Cyclone PCB/FPGA_DENDY.sch (EAGLE design)
At the start: 172 parts, among them CN1 DENDY60PINSLOT, IC1 EP2C5T144, J9 BYPASS, Q1 14.318 MHz, Q2 17.734 MHz, U1 SN74LVC8T245, U10 OPA2134U, U11 SN74LVC2G34DBVR, U13 SN74LVC1G240DBVR, U14 SN74LVC2G34DBVR, U15 SN74LVC1G240DBVR, U16 SN74LVC2G04DBVR, U19 SN74LVC1G125DBVR, U2 SN74LVCH16T245DGGR, U3 SN74LVCH16T245DGGR, U4 74LS373WMSO20, U5 EPCS4, U6 SN74LVC1G240DBVR, U7 THS7374IPWR, U8 SN74LVC1G240DBVR, U9 74LVC1G04GV, X1 057-010-1, X2 JOYPAD1, X3 9V, X4 JOYPAD2

Commit message: Add files via upload
Parts:
- removed C62: 0.1uF, rcl_my:C-EUC0805
- removed C63: 0.1uF, rcl_my:C-EUC0603
- removed IC1: EP2C5T144, EP2C5T144:EP2C5T144
- removed R61: 510, rcl:R-EU_R0805
- removed R63: 1k, rcl:R-EU_R0805
- removed R65: 10k, rcl:R-EU_R0805
- removed R67: 10, rcl:R-EU_R0805
- added C10: 0.1uF, rcl_my:C-EUC0805
- added C26: 1uF, rcl_my:C-EUC0805
- added R10: 51, rcl:R-EU_R0805
- added R30, R43: 2k, rcl:R-EU_R0805
- added R42: 10k, rcl:R-EU_R0805
- added U17: OPA2134U, burr-brown:OPA2134U
- C1: device rcl_my:C-EUC0603 -> rcl_my:C-EUC0805
- C11: value 22uF -> 0.1uF; device rcl_my:C-EUC0603 -> rcl_my:C-EUC0805
- C12, C36, C57: value 1000 -> 0.1uF
- C13: value 0.01uF -> 0.1uF
- C19, C20: value 0.1uF -> 1uF
- C28, C30: value 1uF -> 0.1uF
- C29: value 1uF -> 100uF; device rcl_my:C-EUC0805 -> rcl_my:CPOL-EU153CLV-0505
- C32: value 0.1uF -> 100uF; device rcl_my:C-EUC0805 -> rcl_my:CPOL-EU153CLV-0505
- C34, C4: value 100uF -> 0.1uF; device rcl_my:CPOL-EU153CLV-0505 -> rcl_my:C-EUC0805
- C37: value 1000 -> 22uF; device rcl_my:C-EUC0805 -> rcl_my:CPOL-EU153CLV-0505
- C39: value 10uF -> 1000
- C40: device rcl_my:C-EUC0805 -> rcl_my:CPOL-EU153CLV-0505
- C42, C45, C47, C48: value 0.1uF -> 1000
- C44, C54: value 10uF -> 0.1uF; device rcl_my:CPOL-EU153CLV-0505 -> rcl_my:C-EUC0805
- C46: value 10uF -> 0.1uF
- C49: value 0.1uF -> 0.01uF
- C50, C52: device rcl_my:C-EUC0805 -> rcl_my:C-EUC0603
- C51: value 0.1uF -> 22uF; device rcl_my:C-EUC0805 -> rcl_my:C-EUC0603
- C55, C61: value 0.1uF -> 10uF
- C56: device rcl_my:CPOL-EU153CLV-0505 -> rcl_my:C-EUC0805
- C58: value 1000 -> 10uF; device rcl_my:C-EUC0805 -> rcl_my:CPOL-EU153CLV-0505
- C59: value 0.1uF -> 10uF; device rcl_my:C-EUC0805 -> rcl_my:CPOL-EU153CLV-0505
- C9: value 22uF -> 0.1uF; device rcl_my:CPOL-EU153CLV-0505 -> rcl_my:C-EUC0805
- R1, R13: value 51 -> 4k7
- R11: value 820 -> 2k
- R12: value 2k -> 4k7
- R14: value 750 -> 4k7
- R15: value 750 -> 287
- R16: value 124 -> 750
- R17: value 287 -> 124
- R18, R21: value 124 -> 287
- R19, R22: value 287 -> 750
- R2: value 2k2 -> 1k
- R20: value 750 -> 124
- R23: value 4.7k -> 124
- R24: value 75 -> 2k
- R26, R28: value 4k7 -> 2k
- R27: value 4k7 -> 1k
- R29: value 4k7 -> 820
- R31: value 4k7 -> 10
- R32: value 1k -> 1,1k
- R33: value 2k -> 510
- R34: value 4k7 -> 4.7k
- R35: value 2k -> 75
- R36: value 1k5 -> 75
- R39: value 75 -> 10k
- R4, R5: value 1k -> 10k
- R40: value 1,1k -> 10k
- R41: value 510 -> 10k
- R44: value 10 -> 1k
- R45, R47: value 10k -> 4k7
- R46: value 10k -> 2k2
- R48: value 10k -> 2k
- R49: value 2k -> 1k5
- R50: value 2k -> 1k
- R51: value 2k -> 10k
- R52: value 2k -> 10
- R54: value 510 -> 1k
- R8: value 10k -> 1k
- R9: value 10k -> 51
- U1: value SN74LVC8T245 -> EP2C5T144; device SnapEDA-Library:SN74LVC8T245 -> EP2C5T144:EP2C5T144
- U10: value OPA2134U -> SN74LVC2G34DBVR; device burr-brown:OPA2134U -> SN74LVC2G34DBVR:SN74LVC2G34DBVR
- U11: value SN74LVC2G34DBVR -> THS7374IPWR; device SN74LVC2G34DBVR:SN74LVC2G34DBVR -> THS7374IPWR:THS7374IPWR
- U14: value SN74LVC2G34DBVR -> SN74LVC1G240DBVR; device SN74LVC2G34DBVR:SN74LVC2G34DBVR -> SN74LVC1G240DBVR:SN74LVC1G240DBVR
- U16: value SN74LVC2G04DBVR -> SN74LVC1G240DBVR; device SN74LVC2G04DBVR:SN74LVC2G04DBVR -> SN74LVC1G240DBVR:SN74LVC1G240DBVR
- U2: value SN74LVCH16T245DGGR -> 74LS373WMSO20; device SN74LVCH16T245DGGR:SN74LVCH16T245DGGR -> 74LS373WM:74LS373WMSO20
- U3: value SN74LVCH16T245DGGR -> SN74LVC8T245; device SN74LVCH16T245DGGR:SN74LVCH16T245DGGR -> SnapEDA-Library:SN74LVC8T245
- U4: value 74LS373WMSO20 -> SN74LVCH16T245DGGR; device 74LS373WM:74LS373WMSO20 -> SN74LVCH16T245DGGR:SN74LVCH16T245DGGR
- U5: value EPCS4 -> SN74LVCH16T245DGGR; device EPCS4:EPCS4 -> SN74LVCH16T245DGGR:SN74LVCH16T245DGGR
- U6: value SN74LVC1G240DBVR -> 74LVC1G04GV; device SN74LVC1G240DBVR:SN74LVC1G240DBVR -> 74LVC1G04GV:74LVC1G04GV
- U7: value THS7374IPWR -> EPCS4; device THS7374IPWR:THS7374IPWR -> EPCS4:EPCS4
- U8: value SN74LVC1G240DBVR -> SN74LVC2G04DBVR; device SN74LVC1G240DBVR:SN74LVC1G240DBVR -> SN74LVC2G04DBVR:SN74LVC2G04DBVR
- U9: value 74LVC1G04GV -> SN74LVC2G34DBVR; device 74LVC1G04GV:74LVC1G04GV -> SN74LVC2G34DBVR:SN74LVC2G34DBVR
- renumbered R62 to R54, R64 to R55, R66 to R56, R68 to R57, U19 to U12
Connections:
- net #CS: now also R38.2; no longer R39.2
- net +3V3: now also U10.VCC, U8.VCC; no longer U11.VCC, U16.VCC
- net +5V: now also C12.2, C13.1, C3.2, C31.1, C32.+, C33.1, C4.2, C5.2, C50.2, C53.1, C54.1, C8.2, C9.2, R1.1, R31.1, R34.1, R39.1, R40.1, R41.1, R42.1, U11.VS+, U16.VCC, U2.VCC, U3.VCCB@1, U3.VCCB@2, U4.VCCA@1, U4.VCCA@2, U5.VCCA@1, U5.VCCA@2; no longer C11.2, C15.2, C32.1, C38.2, C4.+, C41.2, C47.2, C5.1, C59.2, C60.1, C61.1, C62.1, C63.2, R23.1, R27.1, R44.1, R45.1, R46.1, R47.1, R48.1, U1.VCCB@1, U1.VCCB@2, U2.VCCA@1, U2.VCCA@2, U3.VCCA@1, U3.VCCA@2, U4.VCC, U7.VS+, U8.VCC
- net /CSO: now also U1.IO2(/CSO), U7./CS; no longer IC1.IO2(/CSO), U5./CS
- net /DENDY: now also R13.2, U1.CLK1; no longer IC1.CLK1, R28.2
- net /IN0: now also U1.IO3, U13./OE; no longer IC1.IO3, U8./OE
- net /IN1: now also U1.IO4, U14./OE, U16./OE; no longer IC1.IO4, U13./OE, U6./OE
- net /IRQ: now also R1.2, U10.IN1; no longer R27.2, U11.IN1
- net /IRQ_FPGA: now also U1.CLK6, U10.OUT1; no longer IC1.CLK6, U11.OUT1
- net /PA13: now also U6.OUT; no longer U9.OUT
- net /PAL: now also R12.2, U1.CLK0; no longer IC1.CLK0, R26.2
- net /PRD: now also U5.2A1; no longer U3.2A1
- net /PRD_FPGA: now also U1.IO25, U5.2B1; no longer IC1.IO25, U3.2B1
- net /PWR: now also U5.2A2; no longer U3.2A2
- net /PWR_FPGA: now also U1.IO24, U5.2B2; no longer IC1.IO24, U3.2B2
- net /RESET: now also C17.2, R14.2, U8.IN1; no longer C31.2, R29.2, U16.IN1
- net /ROMSEL: now also U9.OUT1; no longer U14.OUT1
- net /RS_FPGA: now also U1.IO37, U9.IN1; no longer IC1.IO37, U14.IN1
- net /VCS_FPGA: now also U1.CLK7, U10.OUT2; no longer IC1.CLK7, U11.OUT2
- net A0: now also U4.2A8; no longer U2.2A8
- net A0_FPGA: now also U1.IO38, U4.2B8; no longer IC1.IO38, U2.2B8
- net A1: now also U4.2A7; no longer U2.2A7
- net A10: now also U4.1A3; no longer U2.1A3
- net A10_FPGA: now also U1.IO50, U4.1B3; no longer IC1.IO50, U2.1B3
- net A11: now also U4.1A1; no longer U2.1A1
- net A11_FPGA: now also U1.IO52, U4.1B1; no longer IC1.IO52, U2.1B1
- net A12: now also U4.1A4; no longer U2.1A4
- net A12_FPGA: now also U1.IO49, U4.1B4; no longer IC1.IO49, U2.1B4
- net A13: now also U4.1A6; no longer U2.1A6
- net A13_FPGA: now also U1.IO47, U4.1B6; no longer IC1.IO47, U2.1B6
- net A14: now also U4.1A8; no longer U2.1A8
- net A14_FPGA: now also U1.IO45, U4.1B8; no longer IC1.IO45, U2.1B8
- net A1_FPGA: now also U1.IO39, U4.2B7; no longer IC1.IO39, U2.2B7
- net A2: now also U4.2A6; no longer U2.2A6
- net A2_FPGA: now also U1.IO35, U4.2B6; no longer IC1.IO35, U2.2B6
- net A3: now also U4.2A5; no longer U2.2A5
- net A3_FPGA: now also U1.IO40, U4.2B5; no longer IC1.IO40, U2.2B5
- net A4: now also U4.2A4; no longer U2.2A4
- net A4_FPGA: now also U1.IO41, U4.2B4; no longer IC1.IO41, U2.2B4
- net A5: now also U4.2A3; no longer U2.2A3
- net A5_FPGA: now also U1.IO42, U4.2B3; no longer IC1.IO42, U2.2B3
- net A6: now also U4.2A2; no longer U2.2A2
- net A6_FPGA: now also U1.IO43, U4.2B2; no longer IC1.IO43, U2.2B2
- net A7: now also U4.2A1; no longer U2.2A1
- net A7_FPGA: now also U1.IO44, U4.2B1; no longer IC1.IO44, U2.2B1
- net A8: now also U4.1A7; no longer U2.1A7
- net A8_FPGA: now also U1.IO46, U4.1B7; no longer IC1.IO46, U2.1B7
- net A9: now also U4.1A5; no longer U2.1A5
- net A9_FPGA: now also U1.IO48, U4.1B5; no longer IC1.IO48, U2.1B5
- net ALE: now also U1.IO17, U2.EN; no longer IC1.IO17, U4.EN
- net ASDO: now also U1.IO1(ASDO), U7.ASDI; no longer IC1.IO1(ASDO), U5.ASDI
- net B: now also R35.2; no longer R24.2
- net B0: now also U1.IO74; no longer IC1.IO74
- net B1: now also U1.IO75; no longer IC1.IO75
- net B2: now also U1.IO76; no longer IC1.IO76
- net B3: now also U1.IO77; no longer IC1.IO77
- net B4: now also U1.IO78; no longer IC1.IO78
- net B5: now also U1.IO79; no longer IC1.IO79
- net CLKN: now also R9.2, U1.CLK3; no longer IC1.CLK3, R1.2
- net CLKP: now also R10.2, U1.CLK2; no longer IC1.CLK2, R13.2
- net CONF_DONE: now also R4.2, U1.CONF_DONE; no longer IC1.CONF_DONE, R6.2
- net CS_FPGA: now also R32.2, U1.IO81; no longer IC1.IO81, R40.2
- net D0: now also U15.Y, U16.Y, U5.1A8; no longer U3.1A8, U6.Y, U8.Y
- net D0_FPGA: now also U1.IO26, U5.1B8; no longer IC1.IO26, U3.1B8
- net D1: now also U5.1A7; no longer U3.1A7
- net D1_FPGA: now also U1.IO27, U5.1B7; no longer IC1.IO27, U3.1B7
- net D2: now also U5.1A6; no longer U3.1A6
- net D2_FPGA: now also U1.IO28, U5.1B6; no longer IC1.IO28, U3.1B6
- net D3: now also U5.1A5; no longer U3.1A5
- net D3_FPGA: now also U1.IO29, U5.1B5; no longer IC1.IO29, U3.1B5
- net D4: now also U5.1A4; no longer U3.1A4
- net D4_FPGA: now also U1.IO30, U5.1B4; no longer IC1.IO30, U3.1B4
- net D5: now also U5.1A3; no longer U3.1A3
- net D5_FPGA: now also U1.IO31, U5.1B3; no longer IC1.IO31, U3.1B3
- net D6: now also U5.1A2; no longer U3.1A2
- net D6_FPGA: now also U1.IO32, U5.1B2; no longer IC1.IO32, U3.1B2
- net D7: now also U5.1A1; no longer U3.1A1
- net D7_FPGA: now also U1.IO33, U5.1B1; no longer IC1.IO33, U3.1B1
- net DATA0: now also U1.DATA0, U7.DATA; no longer IC1.DATA0, U5.DATA
- net DB_DIR: now also U1.IO34, U5.1DIR; no longer IC1.IO34, U3.1DIR
- net DCLK: now also U1.DCLK, U7.DCLK; no longer IC1.DCLK, U5.DCLK
- net DMC: now also C49.2, R29.2, R30.1, R44.1, R48.1; no longer C13.2, R11.2, R12.1, R32.1, R35.1
- net DMC_PWM: now also R29.1, U1.IO59; no longer IC1.IO59, R11.1
- net EMPH_B: now also R16.1, U1.IO80; no longer IC1.IO80, R15.1
- net EMPH_G: now also R19.1, U1.IO73; no longer IC1.IO73, R14.1
- net EMPH_R: now also R22.1, U1.IO66; no longer IC1.IO66, R20.1
- net G: now also R36.2; no longer R37.2
- net G0: now also U1.IO67; no longer IC1.IO67
- net G1: now also U1.IO68; no longer IC1.IO68
- net G2: now also U1.IO69; no longer IC1.IO69
- net G3: now also U1.IO70; no longer IC1.IO70
- net G4: now also U1.IO71; no longer IC1.IO71
- net G5: now also U1.IO72; no longer IC1.IO72
- net GND: now also C10.1, C13.2, C2.1, C21.1, C26.2, C27.2, C28.2, C29.-, C3.1, C31.2, C32.-, C34.2, C35.2, C37.-, C38.2, C39.2, C4.1, C41.2, C42.2, C44.2, C47.2, C5.1, C54.2, C57.1, C6.1, C7.1, C8.1, C9.1, R15.1, R18.1, R21.1, R24.2, R28.1, R30.2, R33.1, R46.2, R7.2, R8.2, U1.GAPLL1, U1.GAPLL2, U1.GND@10, U1.GND@11, U1.GND@12, U1.GND@13, U1.GND@14, U1.GND@18, U1.GND@19, U1.GND@20, U1.GND@21, U1.GND@22, U1.GND@23, U1.GND@7, U1.GND@8, U1.GND@9, U1.GPLL1@1, U1.GPLL1@2, U1.GPLL2@1, U1.GPLL2@2, U1.MSEL0, U1.MSEL1, U10.GND, U11.DISABLE, U17A.V-, U2./OE, U2.GND, U3./OE, U4.1DIR, U4.2DIR, U4.GND@1, U4.GND@2, U4.GND@3, U4.GND@4, U4.GND@5, U4.GND@6, U4.GND@7, U4.GND@8, U5.2!OE, U5.2DIR, U5.GND@1, U5.GND@2, U5.GND@3, U5.GND@4, U5.GND@5, U5.GND@6, U5.GND@7, U5.GND@8; no longer C13.1, C2.2, C21.2, C27.1, C28.1, C29.2, C3.2, C31.1, C32.2, C34.-, C35.1, C37.2, C38.1, C4.-, C41.1, C42.1, C47.1, C5.2, C55.2, C57.2, C58.2, C59.1, C6.2, C62.2, C63.1, C7.2, C8.2, C9.-, IC1.GAPLL1, IC1.GAPLL2, IC1.GND@1, IC1.GND@10, IC1.GND@11, IC1.GND@12, IC1.GND@13, IC1.GND@14, IC1.GND@18, IC1.GND@19, IC1.GND@2, IC1.GND@20, IC1.GND@21, IC1.GND@22, IC1.GND@23, IC1.GND@3, IC1.GND@7, IC1.GND@8, IC1.GND@9, IC1.GPLL1@1, IC1.GPLL1@2, IC1.GPLL2@1, IC1.GPLL2@2, IC1.MSEL0, IC1.MSEL1, R12.2, R17.1, R19.1, R2.2, R22.1, R25.2, R3.2, R41.1, R49.1, R9.2, U1./OE, U10A.V-, U2.1DIR, U2.2DIR, U2.GND@1, U2.GND@2, U2.GND@3, U2.GND@4, U2.GND@5, U2.GND@6, U2.GND@7, U2.GND@8, U3.2!OE, U3.2DIR, U3.GND@4, U3.GND@5, U3.GND@6, U3.GND@7, U3.GND@8, U4./OE, U4.GND, U5.GND, U7.DISABLE
- net JOYDATA1: now also R39.2, U15.A; no longer R48.2, U8.A
- net JOYDATA2: now also R41.2, U16.A; no longer R47.2, U6.A
- net LCH: now also C59.-; no longer C44.-
- net LE_FPGA: now also U1.IO7; no longer IC1.IO7
- net M2: now also U4.1A2; no longer U2.1A2
- net M2_FPGA: now also U1.IO51, U14.A, U4.1B2; no longer IC1.IO51, U15.A, U2.1B2
- net N$1: now also C55.1, R43.2, R44.2, R45.2; no longer C39.1, R31.2, R32.2, R33.2
- net N$10: now also U3.A1; no longer U1.A1
- net N$12: now also U3.A2; no longer U1.A2
- net N$13: now also U3.A3; no longer U1.A3
- net N$14: now also R16.2, R17.1; no longer R15.2, R16.1
- net N$17: now also U3.A4; no longer U1.A4
- net N$19: now also R26.2, R27.1; no longer R51.2, R53.1
- net N$2: now also R10.1; no longer R13.1
- net N$24: now also R19.2, R20.1; no longer R14.2, R18.1
- net N$30: now also C56.1, R47.2, R48.2, R49.2; no longer C40.1, R34.2, R35.2, R36.2
- net N$31: now also U3.A5; no longer U1.A5
- net N$32: now also U3.A6; no longer U1.A6
- net N$34: now also R22.2, R23.1; no longer R20.2, R21.1
- net N$37: now also C58.+, R52.2; no longer C43.+, R67.2
- net N$38: now also R20.2, U11.CH2_IN; no longer R19.2, U7.CH2_IN
- net N$4: now also C55.2, U17A.+IN; no longer C39.2, U10A.+IN
- net N$42: now also R50.2, R51.1, U17A.-IN; no longer R63.2, R65.1, U10A.-IN
- net N$43: now also R51.2, R52.1, U17A.OUT; no longer R65.2, R67.1, U10A.OUT
- net N$44: now also U17B.OUT; no longer U10B.OUT
- net N$45: now also U17B.-IN; no longer U10B.-IN
- net N$5: now also C56.2, U17B.+IN; no longer C40.2, U10B.+IN
- net N$50: now also R31.2; no longer R44.2
- net N$53: now also R23.2, U11.CH3_IN; no longer R22.2, U7.CH3_IN
- net N$55: now also C14.2, C15.2, U1.VCCIO1@1, U1.VCCIO1@2, U1.VCCIO1@3; no longer C17.2, C18.2, IC1.VCCIO1@1, IC1.VCCIO1@2, IC1.VCCIO1@3
- net N$56: now also R34.2, U11.BYPASS; no longer R23.2, U7.BYPASS
- net N$58: now also R15.2, U11.CH1_IN; no longer R16.2, U7.CH1_IN
- net N$6: now also R9.1; no longer R1.1
- net N$61: now also U3.A7; no longer U1.A7
- net N$62: now also R32.1, R33.2, U11.CH4_IN; no longer R40.1, R41.2, U7.CH4_IN
- net N$63: now also R11.1; no longer R50.1
- net N$64: now also R35.1, U11.CH1_OUT; no longer R24.1, U7.CH1_OUT
- net N$65: now also R36.1, U11.CH2_OUT; no longer R37.1, U7.CH2_OUT
- net N$66: now also R37.1, U11.CH3_OUT; no longer R38.1, U7.CH3_OUT
- net N$67: now also R38.1, U11.CH4_OUT; no longer R39.1, U7.CH4_OUT
- net N$68: now also R28.2; no longer R49.2
- net N$7: now also C59.+; no longer C44.+
- net N$9: now also U3.A0; no longer U1.A0
- net NCE: now also R7.1, U1.NCE; no longer IC1.NCE, R9.1
- net NCONFIG: now also R6.1, U1.NCONFIG; no longer IC1.NCONFIG, R8.1
- net NSTATUS: now also R5.1, U1.NSTATUS; no longer IC1.NSTATUS, R7.1
- net PA0: now also U2.Q8; no longer U4.Q8
- net PA1: now also U2.Q6; no longer U4.Q6
- net PA10: now also U5.2A5; no longer U3.2A5
- net PA10_FPGA: now also U1.IO21, U5.2B5; no longer IC1.IO21, U3.2B5
- net PA11: now also U5.2A6; no longer U3.2A6
- net PA11_FPGA: now also U1.IO20, U5.2B6; no longer IC1.IO20, U3.2B6
- net PA12: now also U5.2A7; no longer U3.2A7
- net PA12_FPGA: now also U1.IO19, U5.2B7; no longer IC1.IO19, U3.2B7
- net PA13: now also U5.2A8, U6.IN; no longer U3.2A8, U9.IN
- net PA13_FPGA: now also U1.IO18, U5.2B8; no longer IC1.IO18, U3.2B8
- net PA2: now also U2.Q4; no longer U4.Q4
- net PA3: now also U2.Q2; no longer U4.Q2
- net PA4: now also U2.Q1; no longer U4.Q1
- net PA5: now also U2.Q3; no longer U4.Q3
- net PA6: now also U2.Q5; no longer U4.Q5
- net PA7: now also U2.Q7; no longer U4.Q7
- net PA8: now also U5.2A3; no longer U3.2A3
- net PA8_FPGA: now also U1.IO23, U5.2B3; no longer IC1.IO23, U3.2B3
- net PA9: now also U5.2A4; no longer U3.2A4
- net PA9_FPGA: now also U1.IO22, U5.2B4; no longer IC1.IO22, U3.2B4
- net PALSEL0: now also U1.IO6; no longer IC1.IO6
- net PALSEL1: now also U1.IO5; no longer IC1.IO5
- net PD0: now also U2.D8, U3.B0; no longer U1.B0, U4.D8
- net PD0_FPGA: now also U1.IO15; no longer IC1.IO15
- net PD1: now also U2.D6, U3.B2; no longer U1.B2, U4.D6
- net PD1_FPGA: now also U1.IO13; no longer IC1.IO13
- net PD2: now also U2.D4, U3.B4; no longer U1.B4, U4.D4
- net PD2_FPGA: now also U1.IO11; no longer IC1.IO11
- net PD3: now also U2.D2, U3.B6; no longer U1.B6, U4.D2
- net PD3_FPGA: now also U1.IO9; no longer IC1.IO9
- net PD4: now also U2.D1, U3.B7; no longer U1.B7, U4.D1
- net PD4_FPGA: now also U1.IO8; no longer IC1.IO8
- net PD5: now also U2.D3, U3.B5; no longer U1.B5, U4.D3
- net PD5_FPGA: now also U1.IO10; no longer IC1.IO10
- net PD6: now also U2.D5, U3.B3; no longer U1.B3, U4.D5
- net PD6_FPGA: now also U1.IO12; no longer IC1.IO12
- net PD7: now also U2.D7, U3.B1; no longer U1.B1, U4.D7
- net PD7_FPGA: now also U1.IO14; no longer IC1.IO14
- net PD_DIR: now also U1.IO16, U3.DIR; no longer IC1.IO16, U1.DIR
- net R: now also R37.2; no longer R38.2
- net R/W: now also U9.OUT2; no longer U14.OUT2
- net R/W_FPGA: now also U1.IO36, U9.IN2; no longer IC1.IO36, U14.IN2
- net R0: now also U1.IO60; no longer IC1.IO60
- net R1: now also U1.IO61; no longer IC1.IO61
- net R2: now also U1.IO62; no longer IC1.IO62
- net R3: now also U1.IO63; no longer IC1.IO63
- net R4: now also U1.IO64; no longer IC1.IO64
- net R5: now also U1.IO65; no longer IC1.IO65
- net RCH: now also C58.-; no longer C43.-
- net RESET: now also U1.CLK4, U4.1!OE, U4.2!OE, U5.1!OE, U8.OUT1; no longer IC1.CLK4, U16.OUT1, U2.1!OE, U2.2!OE, U3.1!OE
- net SCK1: now also R40.2, U13.Y; no longer R45.2, U15.Y
- net SCK2: now also R42.2, U14.Y; no longer R46.2, U13.Y
- net SND: now also R43.1, R49.1; no longer R33.1, R36.1
- net SND0: now also U1.IO53; no longer IC1.IO53
- net SND1: now also U1.IO54; no longer IC1.IO54
- net SND2: now also U1.IO55; no longer IC1.IO55
- net SND3: now also U1.IO56; no longer IC1.IO56
- net SND4: now also R26.1, U1.IO57; no longer IC1.IO57, R51.1
- net SND5: now also R25.1, U1.IO58; no longer IC1.IO58, R52.1
- net SND_DAC: now also C48.2, R24.1, R25.2, R27.2; no longer C12.2, R25.1, R52.2, R53.2
- net SND_EXT: now also R45.1, R46.1, R47.1; no longer R2.1, R31.1, R34.1
- net TCK: now also R8.1, U1.TCK; no longer IC1.TCK, R3.1
- net TDI: now also R2.1, U1.TDI; no longer IC1.TDI, R4.1
- net TDO: now also U1.TDO; no longer IC1.TDO
- net TMS: now also R3.1, U1.TMS; no longer IC1.TMS, R5.1
- net VA10: now also U8.IN2; no longer U16.IN2
- net VA10_FPGA: now also U1.CLK5, U8.OUT2; no longer IC1.CLK5, U16.OUT2
- net VAPLL1: now also C38.1, C39.1, C40.+, U1.VAPLL1; no longer C55.1, C56.+, C58.1, IC1.VAPLL1
- net VAPLL2: now also C41.1, C42.1, C43.+, U1.VAPLL2; no longer C53.1, C54.+, C57.1, IC1.VAPLL2
- net VCC: now also C29.+, C30.1, C57.2, R11.2, R53.1, U17A.V+; no longer C33.1, C34.+, C42.2, R50.2, R61.1, U10A.V+
- net VCCINT: now also C19.2, C20.2, C26.1, C27.1, C36.1, C37.+, U1.VCCINT@1, U1.VCCINT@2, U1.VCCINT@3, U1.VCCINT@4, U1.VPLL1, U1.VPLL2; no longer C27.2, C28.2, C29.1, C30.1, C8.1, C9.+, IC1.VCCINT@1, IC1.VCCINT@2, IC1.VCCINT@3, IC1.VCCINT@4, IC1.VPLL1, IC1.VPLL2
- net VCCIO: now also C10.2, C11.2, C18.2, C2.2, C21.2, C28.1, C34.1, C35.1, C44.1, C45.1, C46.1, C47.1, C6.2, C7.2, R12.1, R13.1, R14.1, R2.2, R3.2, R4.1, R6.2, U1.VCCIO2@1, U1.VCCIO2@2, U1.VCCIO2@3, U1.VCCIO3@1, U1.VCCIO3@2, U1.VCCIO3@3, U1.VCCIO4@1, U1.VCCIO4@2, U1.VCCIO4@3, U3.VCCA, U4.VCCB@1, U4.VCCB@2, U5.VCCB@1, U5.VCCB@2, U7.VCC@1, U7.VCC@2, U7.VCC@3; no longer C14.2, C19.2, C2.1, C20.2, C21.1, C3.1, C35.2, C36.1, C37.1, C48.2, C49.2, C50.2, C6.1, C7.1, IC1.VCCIO2@1, IC1.VCCIO2@2, IC1.VCCIO2@3, IC1.VCCIO3@1, IC1.VCCIO3@2, IC1.VCCIO3@3, IC1.VCCIO4@1, IC1.VCCIO4@2, IC1.VCCIO4@3, R26.1, R28.1, R29.1, R4.2, R6.1, R7.2, R8.2, U1.VCCA, U2.VCCB@1, U2.VCCB@2, U3.VCCB@1, U3.VCCB@2, U5.VCC@1, U5.VCC@2, U5.VCC@3
- net VPPL3: now also C60.1, C61.1, R50.1, R53.2; no longer C45.1, C46.1, R61.2, R63.1
- net VRAMSC: now also U10.IN2; no longer U11.IN2
Other:
- moved on the sheet: C1, C11, C12, C13, C14, C15, C16, C17, C18, C19, C2, C20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

Commit message: Add files via upload
Parts:
- removed RN15: 1k, resistor-dil:4R-N0603-ARC
- added RN11: 2k, resistor-dil:4R-N0603-ARC
- RN1: value 2k -> 33
- RN10: value 4k7 -> 1k
- RN12: value 33 -> 2k
- RN13: value 33 -> 1k
- RN14: value 2k -> 4k7
- RN2: value 1k -> 33
- RN4, RN7: value 2k -> 1k
- RN5, RN8: value 1k -> 2k
- renumbered Q1 to XO1, Q2 to XO2
Connections:
- removed net +3V3: U10.VCC, U8.VCC
- removed net N$55: C14.2, C15.2, C16.2, U1.VCCIO1@1, U1.VCCIO1@2, U1.VCCIO1@3
- net B0: now also RN5C.2; no longer RN9C.2
- net B1: now also RN5D.2; no longer RN9D.2
- net B2: now also RN3A.2; no longer RN7A.2
- net B3: now also RN3B.2; no longer RN7B.2
- net B4: now also RN3C.2; no longer RN7C.2
- net B5: now also RN3D.2; no longer RN7D.2
- net G0: now also RN8C.2; no longer RN6C.2
- net G1: now also RN8D.2; no longer RN6D.2
- net G2: now also RN6A.2; no longer RN4A.2
- net G3: now also RN6B.2; no longer RN4B.2
- net G4: now also RN6C.2; no longer RN4C.2
- net G5: now also RN6D.2; no longer RN4D.2
- net GND: now also C40.-, C43.-, RN14A.1, RN14D.1; no longer RN10A.1, RN10D.1
- net N$10: now also RN1B.2; no longer RN12B.2
- net N$12: now also RN1C.2; no longer RN12C.2
- net N$13: now also RN1D.2; no longer RN12D.2
- net N$14: now also RN3D.1, RN4D.2; no longer RN7D.1, RN8D.2
- net N$16: now also RN3C.1, RN4C.2, RN4D.1; no longer RN7C.1, RN8C.2, RN8D.1
- net N$17: now also RN2A.2; no longer RN13A.2
- net N$18: now also RN3B.1, RN4B.2, RN4C.1; no longer RN7B.1, RN8B.2, RN8C.1
- net N$19: now also RN13D.1; no longer RN15D.1
- net N$23: now also RN3A.1, RN4A.2, RN4B.1; no longer RN7A.1, RN8A.2, RN8B.1
- net N$24: now also RN6D.1, RN7D.2; no longer RN4D.1, RN5D.2
- net N$25: now also RN6C.1, RN7C.2, RN7D.1; no longer RN4C.1, RN5C.2, RN5D.1
- net N$26: now also RN6B.1, RN7B.2, RN7C.1; no longer RN4B.1, RN5B.2, RN5C.1
- net N$27: now also RN4A.1, RN5A.1, RN5B.1, RN5D.1; no longer RN8A.1, RN9A.1, RN9B.1, RN9D.1
- net N$28: now also RN6A.1, RN7A.2, RN7B.1; no longer RN4A.1, RN5A.2, RN5B.1
- net N$29: now also RN5A.2, RN5B.2, RN5C.1; no longer RN9A.2, RN9B.2, RN9C.1
- net N$31: now also RN2B.2; no longer RN13B.2
- net N$32: now also RN2C.2; no longer RN13C.2
- net N$33: now also RN7A.1, RN8A.1, RN8B.1, RN8D.1; no longer RN5A.1, RN6A.1, RN6B.1, RN6D.1
- net N$34: now also RN10D.2, RN9D.1; no longer RN1D.1, RN2D.2
- net N$35: now also RN10C.2, RN10D.1, RN9C.1; no longer RN1C.1, RN2C.2, RN2D.1
- net N$36: now also RN8A.2, RN8B.2, RN8C.1; no longer RN6A.2, RN6B.2, RN6C.1
- net N$39: now also RN10B.2, RN10C.1, RN9B.1; no longer RN1B.1, RN2B.2, RN2C.1
- net N$4: now also RN14C.1, RN14D.2; no longer RN10C.1, RN10D.2
- net N$40: now also RN10A.2, RN10B.1, RN9A.1; no longer RN1A.1, RN2A.2, RN2B.1
- net N$41: now also RN10A.1, RN11A.1, RN11B.1, RN11D.1; no longer RN2A.1, RN3A.1, RN3B.1, RN3D.1
- net N$5: now also RN14A.2, RN14B.1; no longer RN10A.2, RN10B.1
- net N$52: now also RN12D.1, RN13C.1, RN13D.2; no longer RN14D.1, RN15C.1, RN15D.2
- net N$54: now also RN12C.1, RN13B.1, RN13C.2; no longer RN14C.1, RN15B.1, RN15C.2
- net N$60: now also RN12B.1, RN13A.1, RN13B.2; no longer RN14B.1, RN15A.1, RN15B.2
- net N$61: now also RN2D.2; no longer RN13D.2
- net N$68: now also RN12A.1, RN13A.2; no longer RN14A.1, RN15A.2
- net N$71: now also RN11A.2, RN11B.2, RN11C.1; no longer RN3A.2, RN3B.2, RN3C.1
- net N$9: now also RN1A.2; no longer RN12A.2
- net PD0_FPGA: now also RN1A.1; no longer RN12A.1
- net PD1_FPGA: now also RN1C.1; no longer RN12C.1
- net PD2_FPGA: now also RN2A.1; no longer RN13A.1
- net PD3_FPGA: now also RN2C.1; no longer RN13C.1
- net PD4_FPGA: now also RN2D.1; no longer RN13D.1
- net PD5_FPGA: now also RN2B.1; no longer RN13B.1
- net PD6_FPGA: now also RN1D.1; no longer RN12D.1
- net PD7_FPGA: now also RN1B.1; no longer RN12B.1
- net R0: now also RN11C.2; no longer RN3C.2
- net R1: now also RN11D.2; no longer RN3D.2
- net R2: now also RN9A.2; no longer RN1A.2
- net R3: now also RN9B.2; no longer RN1B.2
- net R4: now also RN9C.2; no longer RN1C.2
- net R5: now also RN9D.2; no longer RN1D.2
- net SND0: now also RN12A.2; no longer RN14A.2
- net SND1: now also RN12B.2; no longer RN14B.2
- net SND2: now also RN12C.2; no longer RN14C.2
- net SND3: now also RN12D.2; no longer RN14D.2
- net VCC: now also RN14B.2, RN14C.2; no longer RN10B.2, RN10C.2
- net VCCIO: now also C14.2, C15.2, C16.2, U1.VCCIO1@1, U1.VCCIO1@2, U1.VCCIO1@3, U10.VCC, U8.VCC
Other:
- moved on the sheet: C1, C17, C2, C3, C32, C33, C34, C35, C36, C37, R1, RN10A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
