File: PCB/Cyclone PCB/FPGA_DENDY.sch (EAGLE design)
At the start: 179 parts, among them CN1 DENDY60PINSLOT, J9 BYPASS, U1 EP2C5T144, U10 SN74LVC2G34DBVR, U11 THS7374IPWR, U12 SN74LVC1G125DBVR, U13 SN74LVC1G240DBVR, U14 SN74LVC1G240DBVR, U15 SN74LVC1G240DBVR, U16 SN74LVC1G240DBVR, U17 OPA2134U, U2 74LS373WMSO20, U3 SN74LVC8T245, U4 SN74LVCH16T245DGGR, U5 SN74LVCH16T245DGGR, U6 74LVC1G04GV, U7 EPCS4, U8 SN74LVC2G04DBVR, U9 SN74LVC2G34DBVR, X1 057-010-1, X2 JOYPAD1, X3 9V, X4 JOYPAD2

Commit message: fix snd_dac
Connections:
- removed net SND: R44.1, R50.1
- net SND_DAC: now also R44.1, R50.1
Changed lines of the file:
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@@
 <setting verticaltext="up"/>
 </settings>
-<grid distance="0.1" unitdist="inch" unit="inch" style="lines" multiple="1" display="yes" altdistance="0.01" altunitdist="inch" altunit="inch"/>
+<grid distance="0.1" unitdist="inch" unit="inch" style="lines" multiple="1" display="no" altdistance="0.01" altunitdist="inch" altunit="inch"/>
 <layers>
 <layer number="1" name="Top" color="4" fill="1" visible="no" active="no"/>
@@
 <junction x="137.16" y="-5.08"/>
 </segment>
+<segment>
+<wire x1="170.18" y1="-53.34" x2="187.96" y2="-53.34" width="0.1524" layer="91"/>
+<label x="172.72" y="-53.34" size="1.778" layer="95"/>
+<pinref part="R44" gate="G$1" pin="1"/>
+</segment>
+<segment>
+<wire x1="170.18" y1="-104.14" x2="187.96" y2="-104.14" width="0.1524" layer="91"/>
+<label x="172.72" y="-104.14" size="1.778" layer="95"/>
+<pinref part="R50" gate="G$1" pin="1"/>
+</segment>
 </net>
 <net name="DMC" class="0">
@@
 </segment>
 </net>
-<net name="SND" class="0">
-<segment>
-<wire x1="170.18" y1="-104.14" x2="187.96" y2="-104.14" width="0.1524" layer="91"/>
-<label x="172.72" y="-104.14" size="1.778" layer="95"/>
-<pinref part="R50" gate="G$1" pin="1"/>
-</segment>
-<segment>
-<wire x1="170.18" y1="-53.34" x2="187.96" y2="-53.34" width="0.1524" layer="91"/>
-<label x="172.72" y="-53.34" size="1.778" layer="95"/>
-<pinref part="R44" gate="G$1" pin="1"/>
-</segment>
-</net>
